File: ZombieDelay.sch (EAGLE design)
At the start: 79 parts, among them IC1 MAX1044, IC2 TL072P, IC3 78L05Z, IC4 78L12Z, Q1 2N5089

Commit message: Making an offshoot pedal Zombie Delay with artwork by Tad Leger
Parts:
- added 3MM: LED3MM, mb_diodes:LED3MM
- DELAY, LEVEL, REPEATS: device mb_pots:POT16MM -> mb_pots:POT16MM_PCB_PADS
Connections:
- new net N$4: 3MM.A, R28.1
- net D: now also 3MM.C
Changed lines of the file:
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@@
 <part name="GND17" library="mb_supply" deviceset="GND" device=""/>
 <part name="GND18" library="mb_supply" deviceset="GND" device=""/>
-<part name="DELAY" library="mb_pots" deviceset="POT" device="16MM" value="B50K"/>
+<part name="DELAY" library="mb_pots" deviceset="POT" device="16MM_PCB_PADS" value="B50K"/>
 <part name="GND19" library="mb_supply" deviceset="GND" device=""/>
 <part name="R10" library="mb_resistors" deviceset="6MM" device=".3" value="22k"/>
@@
 <part name="C41" library="mb_caps-box" deviceset="072X045" device="2" value="1uF"/>
 <part name="GND29" library="mb_supply" deviceset="GND" device=""/>
-<part name="LEVEL" library="mb_pots" deviceset="POT" device="16MM" value="B50K"/>
-<part name="REPEATS" library="mb_pots" deviceset="POT" device="16MM" value="B50K"/>
+<part name="LEVEL" library="mb_pots" deviceset="POT" device="16MM_PCB_PADS" value="B50K"/>
+<part name="REPEATS" library="mb_pots" deviceset="POT" device="16MM_PCB_PADS" value="B50K"/>
 <part name="GND30" library="mb_supply" deviceset="GND" device=""/>
 <part name="GND31" library="mb_supply" deviceset="GND" device=""/>
@@
 <part name="R28" library="mb_resistors" deviceset="6MM" device=".3" value="4k7"/>
 <part name="V3" library="mb_supply" deviceset="+9V" device=""/>
+<part name="3MM" library="mb_diodes" deviceset="LED" device="3MM"/>
+<part name="D5" library="mb_supply" deviceset="D" device=""/>
 </parts>
 <sheets>
@@
 <attribute name="VALUE" x="12.319" y="102.489" size="1.778" layer="96" rot="R90"/>
 </instance>
+<instance part="3MM" gate="G$1" x="43.18" y="104.14" smashed="yes" rot="R180">
+<attribute name="NAME" x="45.212" y="107.696" size="1.778" layer="95" rot="R180"/>
+</instance>
+<instance part="D5" gate="D" x="50.8" y="104.14" smashed="yes">
+<attribute name="VALUE" x="55.88" y="103.124" size="1.778" layer="96" rot="R90"/>
+</instance>
 </instances>
 <busses>
@@
 <wire x1="-5.08" y1="88.9" x2="-7.62" y2="88.9" width="0.1524" layer="91"/>
 </segment>
+<segment>
+<pinref part="D5" gate="D" pin="D"/>
+<pinref part="3MM" gate="G$1" pin="C"/>
+<wire x1="48.26" y1="104.14" x2="45.72" y2="104.14" width="0.1524" layer="91"/>
+</segment>
 </net>
 <net name="+9V" class="0">
@@
 </segment>
 </net>
+<net name="N$4" class="0">
+<segment>
+<pinref part="3MM" gate="G$1" pin="A"/>
+<pinref part="R28" gate="G$1" pin="1"/>
+<wire x1="38.1" y1="104.14" x2="33.02" y2="104.14" width="0.1524" layer="91"/>
+</segment>
+</net>
