File: ZombieDelay.brd (EAGLE design)
At the start: 82.2 x 55.9 mm, 80 parts, among them IC1 MAX1044, IC2 TL072P, IC3 78L05Z, IC4 78L12Z, Q1 2N5089

Commit message: Updated to include larger regulators
Parts:
- IC3: value 78L05Z -> 7805T; device mb_regulators:TO92 -> mb_regulators:TO220H
- IC4: value 78L12Z -> 7812T; device mb_regulators:TO92 -> mb_regulators:TO220H
- moved IC4 6.91 mm to (70.3, 22.4)
- moved IC3 6.75 mm to (75.5, 24.7)
- moved R1 6.34 mm to (64.7, 39.8), turned to 180 degrees
- moved C37 5.71 mm to (60.7, 47.1)
- moved C4 1.48 mm to (69.7, 16.7)
- moved R6 1.05 mm to (73.1, 41.7)
Routing:
- net N$41: track 42.0 -> 50.0 mm
- net C: track 47.5 -> 52.0 mm
- net B: track 125.9 -> 122.2 mm
- net N$46: track 8.06 -> 11.5 mm
- net N$49: track 16.4 -> 19.8 mm
- net N$9: track 23.2 -> 26.2 mm
- net N$6: track 94.9 -> 97.2 mm
- net N$13: track 18.3 -> 16.7 mm
- net N$8: track 137.2 -> 136.1 mm
- net N$1: track 39.1 -> 38.1 mm
- net N$11: track 89.2 -> 89.9 mm
Other:
- board text added: "Xenocoder Zombie Delay v1.1 2025 02"
- board text removed: "Xenocoder Zombie Delay v1.0 2020 04"
